File: CurrentController.brd (EAGLE design)
At the start: 160 x 100 mm, 135 parts, among them CN1 220uF, CN2 10uF, CN3 47uF, IC1 LM340S-12, IC2 L7912, IC3 TS514, IC4 AD8676, IC5 MEGA8-AI, IC6 78L05F, IC7 AD8676, T1 PVG3A, X1 1-227161-7, X2 1-227161-7, X3 1-227161-7

Commit message: Working on re-routing; about to add feed forward
Parts:
- removed CD7: 100nF, rcl:C0402K
- removed CL10, CL11, CL9: 10nF, rcl:C0402K
- removed CN2, CP2, CR9: 10uF, rcl:C0805K
- removed J2: (no value), 19inch:VG64PD
- removed JP2: (no value), pinhead:1X05
- removed JP3: (no value), pinhead:1X02
- removed JP4: (no value), pinhead:1X07
- removed JP5: (no value), pinhead:1X07-SMD
- removed LN1, LP1: SDR1005-101K, misc-ics:SDR1000-INDUCT
- removed R10, R25, R9: 10k, rcl:R0402
- removed R27: 0R, rcl:R0402
- removed R30, R31, R32, R33, R34, R35: 100R, rcl:R0402
- removed T1: PVG3A, misc-ics:PVG3A
- removed VREG1: TPS7A470, misc-ics:S-PVQFN-N20
- removed X1, X2, X3: 1-227161-7, con-coax:AMP_227161
- added C10, C11, C12, C13, C14, C15, C16: 10uF, jqi_passives:C_MLCC_0805
- added C17: 1uF, jqi_passives:C_MLCC_0603
- added CUR, MOD_IN, MON: BNC-H, connector-jqi:BNC90
- added D1: Schottky, diode:SOD523
- added ENC, LCD: (no value), mcu-accessories:ML08
- added F1, F2, F3, F4, F5, F6, F7, F8: (no value), jqi_passives:R_0805
- added J1: (no value), connector-jqi:VG64-CUTOUT
- added L1, L2: 100uH, jqi_passives:COILCRAFT_MSS1583
- added R6: 0R, jqi_passives:R_1206
- added U1: TPS7A470, regulator-jqi:S-PVQFN-N20
- C1: device rcl:C1206K -> jqi_passives:C_POL_1206
- C2, C3, CD3, CL12, CL8: device rcl:C0402K -> jqi_passives:C_MLCC_0402
- C27, C28, C29, CL1, CL2, CL3, CL4, CL5, CL6, MC1: device rcl:C0402K -> jqi_passives:C_MLCC_0603
- C30, C31: value 100nF -> 10nF; device rcl:C0402K -> jqi_passives:C_MLCC_0603
- C4, C5, C6, C7, C8, C9, CR1, CR12, CR2, CR3, CR4, CR5, CR6, CR8: device rcl:C0805K -> jqi_passives:C_MLCC_0805
- MON1, R1, R100, R12, R14, R15, R16, R17, R18, R19, R2, R21, R22, R23, R24, R26, R36, R37, R38, R39, R4, R40, R41, R42, R43, R44, R45, R46, R47, R48, R49, R5, R50, R51, R52, R53, R54: device rcl:R0402 -> jqi_passives:R_0603
- MR1, MR2, MR3, MR4, MR5, MR6, MR7, MR8, MR9: device rcl:R0805 -> jqi_passives:R_0805
- R20: device rcl:R0402 -> jqi_passives:R_0805
- R3, R7, R8: value 10k -> 0R; device rcl:R0402 -> jqi_passives:R_1206
- RJH1: value 0R -> 0R_DNP; device rcl:R0402 -> jqi_passives:R_0402
- SV2: device con-lstb:MA08-2 -> connector-jqi:MA08-2
- moved C29 151.7 mm to (241.0, 114.3), turned to 0 degrees
- moved IC6 144.8 mm to (238.3, 111.5), turned to 90 degrees
- moved R36 111.2 mm to (182.6, 8.13)
- moved R37 111.2 mm to (181.9, 6.35)
- moved R12 111.2 mm to (184.4, 8.13)
- moved VREFIC 111.2 mm to (186.9, -0.51)
- moved C3 109.5 mm to (47.2, -68.8)
- moved C30 109.5 mm to (70.4, -56.9)
- moved C4 109.5 mm to (52.6, -68.8)
- moved C7 109.5 mm to (52.6, -68.8)
- moved CL2 109.5 mm to (44.2, -71.9)
- moved CL8 109.5 mm to (60.5, -64.5)
- moved CR1 109.5 mm to (49.4, -78.2)
- moved CR2 109.5 mm to (42.4, -73.9)
- moved CR8 109.5 mm to (63.2, -71.9)
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Connections:
- net N$6 renamed DC_OUT
- removed net +12V: BUF1.8, C29.1, C30.1, CL12.1, CL2.1, CL3.1, CL5.1, CR12.1, CR2.1, CR3.1, CR5.1, IC1.3, IC3.4, IC4.8, IC6.3, IC7.8, R15.1, VREFIC.3, VREG1.15, VREG1.16
- removed net +5V: CD7.1, CL9.1, CR9.1, IC5.18, IC5.4, IC5.6, IC6.1, JP5.2, JP6.1, R10.1, R100.2, R21.1, R25.2, R3.1, R9.1, SV1.2
- removed net -12V: BUF1.4, C31.1, CL1.1, CL4.1, CL6.1, CR1.1, CR4.1, CR6.1, IC2.3, IC3.11, IC4.4, IC7.4, R22.2, R37.1, VREFIC.4
- removed net D2: CL10.1, IC5.32, R7.2
- removed net D3: CL11.1, IC5.1, R8.2
- removed net D5: IC5.9, R26.1, R27.2
- removed net D8: IC5.12, JP2.4, R10.2
- removed net D9: IC5.13, R46.2
- removed net ENABLE: R27.1, VREG1.13
- removed net N$22: R14.1, R15.2, R16.1
- removed net N$53: JP4.1, R32.2
- removed net N$54: JP4.2, R33.2
- removed net N$55: JP4.3, R34.2
- removed net N$56: JP4.4, R35.2
- removed net VOUT: IC4.5, MR6.2, MR7.1, RJH1.2
- new net CURR_OUT: CUR.1, LOUT1.2, RJH1.P$1
- new net DAC_CS: IC5.13, R46.P$2
- new net ENC_A: ENC.8, IC5.32
- new net ENC_B: ENC.6, IC5.1
- new net ENC_SW: ENC.4, IC5.12
- new net LCD_CS: LCD.6
- new net LCD_RS: LCD.7
- new net LCD_RST: LCD.8
- new net MOD_OUT: IC4.5, MR6.P$2, MR7.P$1, RJH1.P$2
- new net N$24: IC2.TAB, R3.P$2
- new net N$26: IC1.1, R6.P$2
- new net N$29: R14.P$1, R15.P$2, R16.P$1
- new net N$30: CN3.-, L2.P$2, R3.P$1, R7.P$1
- new net N$50: CL1.P$1, CR1.P$1, F6.P$1, IC7.4
- new net N$52: CL2.P$1, CR2.P$1, F5.P$1, IC7.8
- new net N$6: CL5.P$1, CR5.P$1, F1.P$1, IC4.8
- new net SW: ENC.7
- new net VCC: C17.P$1, ENC.1, IC5.18, IC5.4, IC5.6, IC6.1, JP6.1, LCD.1, R100.P$2, R21.P$1, SV1.2
- new net VREG_EN: IC5.9, R26.P$1, U1.13
- new net VSS: C17.P$2, C29.P$2, ENC.2, IC5.21, IC5.3, IC5.5, IC6.2, IC6.2@1, JP1.1, JP1.2, JP6.3, LCD.2, LCD.4, SV1.6
- net +15V: now also J1.A31, J1.C31, L1.P$1; no longer CP2.1, J2.A31, J2.C31, LP1.P$1
- net -15V: now also J1.A30, J1.C30, L2.P$1; no longer CN2.2, J2.A30, J2.C30, LN1.P$1
- net A4: now also R14.P$2; no longer R14.2
- net A5: now also R17.P$2; no longer R17.2
- net A6: now also R18.P$2; no longer R18.2
- net A7: now also R19.P$2; no longer R19.2
- net D4: no longer JP3.2, R25.1
- net D6: no longer R31.1
- net D7: no longer R30.1
- net DACG: now also CD3.P$2, CL8.P$2, CR8.P$2, R39.P$1, R43.P$1, R47.P$2; no longer CD3.2, CL8.2, CR8.2, R39.1, R43.1, R47.2
- net DCLK: now also R41.P$1; no longer R41.1
- net DCS: now also R49.P$2; no longer R49.2
- net DDATA: now also R45.P$1; no longer R45.1
- net DTR: now also C28.P$1; no longer C28.1
- net GND: now also C1.P$2, C10.P$2, C11.P$2, C12.P$2, C13.P$2, C14.P$2, C15.P$2, C16.P$2, C2.P$2, C27.P$2, C30.P$2, C31.P$2, CL1.P$2, CL12.P$2, CL2.P$2, CL3.P$2, CL4.P$2, CL5.P$2, CL6.P$2, CR1.P$2, CR12.P$2, CR2.P$2, CR3.P$2, CR4.P$2, CR5.P$2, CR6.P$2, CUR.2, J1.A1, J1.C1, MOD_IN.2, MON.2, MR1.P$1, MR5.P$2, R16.P$2, R20.P$1, R24.P$2, R40.P$1, R44.P$1, R48.P$2, R54.P$2, U1.17, U1.18, U1.19, U1.2, U1.7, U1.EXP; no longer C1.2, C2.2, C27.2, C29.2, C30.2, C31.2, CD7.2, CL1.2, CL10.2, CL11.2, CL12.2, CL2.2, CL3.2, CL4.2, CL5.2, CL6.2, CL9.2, CN2.1, CP2.2, CR1.2, CR12.2, CR2.2, CR3.2, CR4.2, CR5.2, CR6.2, CR9.2, IC5.21, IC5.3, IC5.5, IC6.2, IC6.2@1, J2.A1, JP1.1, JP1.2, JP2.2, JP2.5, JP3.1, JP4.5, JP4.6, JP4.7, JP5.1, JP5.5, JP5.7, JP6.3, MR1.1, MR5.2, R16.2, R20.1, R24.2, R40.1, R44.1, R48.2, R54.2, SV1.6, T1.P$1, VREG1.7, X1.2, X2.2, X3.2
- net MODIN_B: now also MOD_IN.1, MR7.P$2, MR8.P$1, R20.P$2; no longer MR7.2, MR8.1, R20.2, X2.1
- net MON: now also MON1.P$1, R51.P$1; no longer MON1.1, R51.1
- net MON_MON: now also MON.1, MON1.P$2, R19.P$1; no longer MON1.2, R19.1, X3.1
- net MOSI: now also LCD.3, R42.P$2; no longer R42.2
- net N$1: now also MR8.P$2, MR9.P$1; no longer MR8.2, MR9.1
- net N$10: now also R1.P$1; no longer R1.1
- net N$11: now also R1.P$2, R2.P$1; no longer R1.2, R2.1
- net N$12: now also R17.P$1, R21.P$2, R22.P$1; no longer R17.1, R21.2, R22.1
- net N$13: now also C3.P$2, R2.P$2; no longer C3.2, R2.2
- net N$14: now also R51.P$2, R52.P$1; no longer R51.2, R52.1
- net N$16: now also R40.P$2, R41.P$2; no longer R40.2, R41.2
- net N$17: now also R53.P$1, R54.P$1; no longer R53.1, R54.1
- net N$18: now also MR1.P$2, MR2.P$2; no longer MR1.2, MR2.2
- net N$19: now also SV2.2, U1.4; no longer SV2.16, VREG1.12
- net N$2: now also R26.P$2; no longer R26.2
- net N$20: now also MR2.P$1, MR3.P$2, MR6.P$1; no longer MR2.1, MR3.2, MR6.1
- net N$21: now also MR5.P$1; no longer MR5.1
- net N$23: now also MC1.P$2, MR4.P$1, MR9.P$2; no longer MC1.2, MR4.1, MR9.2
- net N$25: now also MC1.P$1, MR3.P$1, MR4.P$2; no longer MC1.1, MR3.1, MR4.2
- net N$27: now also SV2.4, U1.5; no longer C2.1, VREG1.14
- net N$28: now also R36.P$1, R37.P$2; no longer R36.1, R37.2
- net N$3: now also IC3.9, R48.P$1, R49.P$1; no longer JP2.1, R7.1, R9.2
- net N$31: now also SV2.6, U1.6; no longer SV2.14, VREG1.11
- net N$32: now also CP3.+, L1.P$2, R6.P$1, R8.P$1; no longer C27.1, IC5.20
- net N$33: now also R18.P$1, R23.P$2, R24.P$1; no longer R18.1, R23.2, R24.1
- net N$34: now also SV2.8, U1.8; no longer SV2.12, VREG1.10
- net N$36: now also BUF1.4, CL4.P$1, CR4.P$1, F4.P$1; no longer JP5.4, R30.2
- net N$37: now also BUF1.8, CL3.P$1, CR3.P$1, F3.P$1; no longer IC3.9, R48.1, R49.1
- net N$38: now also C10.P$1, C30.P$1, F7.P$2, IC3.4; no longer JP5.6, R31.2
- net N$39: now also U1.9; no longer VREG1.9
- net N$4: now also R52.P$2; no longer R52.2
- net N$40: now also R38.P$1, R39.P$2; no longer R38.1, R39.2
- net N$41: now also SV2.12, U1.10; no longer SV2.8, VREG1.8
- net N$42: now also R42.P$1, R43.P$2; no longer R42.1, R43.2
- net N$43: now also SV2.14, U1.11; no longer SV2.6, VREG1.6
- net N$44: now also SV2.16, U1.12; no longer SV2.4, VREG1.5
- net N$45: now also C2.P$1, U1.14; no longer SV2.2, VREG1.4
- net N$46: now also C11.P$1, C31.P$1, F8.P$2, IC3.11; no longer JP5.3, T1.P$2
- net N$47: now also R44.P$2, R45.P$2; no longer R44.2, R45.2
- net N$48: now also C6.P$2, C9.P$2, R50.P$1; no longer C6.2, C9.2, R50.1
- net N$49: now also R46.P$1, R47.P$1; no longer R46.1, R47.1
- net N$5: now also C27.P$1, IC5.20; no longer JP2.3, R3.2, R8.1
- net N$7: now also CL6.P$1, CR6.P$1, F2.P$1, IC4.4; no longer LOUT1.2, RJH1.1, X1.1
- net N$8: now also C4.P$2, C7.P$2, R4.P$1, R5.P$2; no longer C4.2, C7.2, R4.1, R5.2
- net N$9: now also C5.P$2, C8.P$2, R5.P$1; no longer C5.2, C8.2, R5.1
- net PC0: no longer R35.1
- net PC1: no longer R34.1
- net PC2: no longer R33.1
- net PC3: no longer R32.1
- net RESET: now also C28.P$2, R100.P$1; no longer C28.2, R100.1
- net SCK: now also LCD.5, R38.P$2; no longer R38.2
- net V+: now also C1.P$1, C29.P$1, CL12.P$1, CR12.P$1, F1.P$2, F3.P$2, F5.P$2, F7.P$1, IC1.3, IC6.3, R15.P$1, R8.P$2, U1.15, U1.16, VREFIC.3; no longer CP3.+, IC1.1, LP1.P$2
- net V-: now also F2.P$2, F4.P$2, F6.P$2, F8.P$1, IC2.3, R22.P$2, R37.P$1, R7.P$2, VREFIC.4; no longer CN3.-, IC2.TAB, LN1.P$2
- net VREF: now also R12.P$1, R36.P$2, R50.P$2; no longer R12.1, R36.2, R50.2
- net VREG: now also C12.P$1, C13.P$1, C14.P$1, C15.P$1, C16.P$1, C3.P$1, C4.P$1, C5.P$1, C6.P$1, C7.P$1, C8.P$1, C9.P$1, CD3.P$1, CL8.P$1, CR8.P$1, R12.P$2, R23.P$1, R53.P$2, U1.1, U1.20, U1.3; no longer C1.1, C3.1, C4.1, C5.1, C6.1, C7.1, C8.1, C9.1, CD3.1, CL8.1, CR8.1, R12.2, R23.1, R53.2, VREG1.1, VREG1.20, VREG1.3
- net VSET: now also R4.P$2; no longer R4.2
Routing:
- net MON_MON: track 249.7 -> 0.00 mm, vias 3 -> 0
- net +12V: track 211.8 -> 0.00 mm, vias 9 -> 0
- net +5V: track 209.7 -> 0.00 mm
- net -12V: track 164.3 -> 0.00 mm, vias 7 -> 0
- net D6: track 123.5 -> 0.00 mm, vias 2 -> 0
- net D7: track 123.1 -> 0.00 mm, vias 2 -> 0
- net PC0: track 107.0 -> 0.00 mm, vias 2 -> 0
- net PC1: track 104.9 -> 0.00 mm, vias 2 -> 0
- net PC2: track 103.2 -> 0.00 mm, vias 2 -> 0
- net PC3: track 101.9 -> 0.00 mm, vias 2 -> 0
- net N$33: track 101.8 -> 0.00 mm, vias 2 -> 0
- net ENABLE: track 86.9 -> 0.00 mm, vias 2 -> 0
- net N$40: track 70.6 -> 0.00 mm, vias 3 -> 0
- net D8: track 70.0 -> 0.00 mm, vias 1 -> 0
- net VREG: track 67.0 -> 0.00 mm, vias 12 -> 0
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- added copper zone on layer 1, net +15V
- added copper zone on layer 1, net -15V
- added copper zone on layer 1, net N$24
- added copper zone on layer 1, net N$30
- added copper zone on layer 1, net N$32
- added copper zone on layer 1, net V+
- added copper zone on layer 1, net V-
- removed copper zone on layer 1, net +12V
- removed copper zone on layer 15, net +12V
- removed copper zone on layer 1, net +5V
- removed copper zone on layer 1, net -12V
- removed copper zone on layer 16, net -12V
- removed copper zone on layer 1, net DACG
- removed copper zone on layer 15, net DACG
- removed copper zone on layer 16, net DACG
- removed copper zone on layer 1, net GND
- removed copper zone on layer 16, net GND
- removed copper zone on layer 2, net GND
- removed copper zone on layer 1, net N$15
- removed copper zone on layer 15, net VREG
- removed copper zone on layer 16, net VREG
Other:
- outline, holes or cut-outs redrawn
- board text added: "+5V"
- board text added: "0.1V"
- board text added: "0.2V"
- board text added: "0.4V"
- board text added: "0.8V"
- board text added: "1.6V"
- board text added: "3.2V"
- board text added: "6.4V"
- board text added: "DTR"
- board text added: "FTDI Header"
- board text added: "ISP Prog"
- board text added: "Normal"
- board text added: "RX"
- board text added: "TX"
- board text added: "Vreg = 1.4V +"
- board text added: "short"
- board text removed: "Contrast"

Commit message: mostly routed, few remaining tweaks
Parts:
- removed BUF1, IC7: AD8676, analog-devices:MSOP08
- removed CD3: 100nF, jqi_passives:C_MLCC_0402
- removed CL8: 10nF, jqi_passives:C_MLCC_0402
- removed CR1, CR2, CR5, CR6, CR8: 10uF, jqi_passives:C_MLCC_0805
- removed F1, F2, F5, F6: (no value), jqi_passives:R_0805
- removed JP6: (no value), pinhead:1X03
- removed R24, R26, R38, R39, R40, R41, R42, R43, R44, R45, R46, R47, R48, R49, R51, R52, R53, R54: 10k, jqi_passives:R_0603
- added BUF, FFWD, U2, U3: AD8676, opamp-jqi:MSOP08
- added C18: (no value), jqi_passives:C_MLCC_0603
- added C19, C20: 1uF, jqi_passives:C_MLCC_0603
- added C21, C25, C26: 10nF, jqi_passives:C_MLCC_0306
- added C22, C23, C32, C33, CD1, CD2: 100nF, jqi_passives:C_MLCC_0603
- added C24: 0.47uF, jqi_passives:C_MLCC_0612
- added D3, D4: Schottky, diode:SOD523
- added F9: 1k_ferrite, jqi_passives:L_FERRITE_0603
- added JP2: (no value), pinhead:1X03
- added JP3: (no value), pinhead:2X08
- added L3: (no value), jqi_passives:R_0805
- added MR10, MR11: 1k, jqi_passives:R_0805
- added R10, R11, R13, R9: 10k, jqi_passives:742_ARRAY
- added R25: 200k, jqi_passives:R_0603
- added T1: 100k, rlc-jqi:3006P
- added U$4: (no value), JQI_Logo:JQI_LOGO_NEGATIVE-SILKSCREEN
- added U$5: WURTH_EMI, mcu-accessories:WURTH_SHIELD
- added U4: NT2006, semiconductor-jqi:HVQFN16
- C10: value 10uF -> 0.47uF; device jqi_passives:C_MLCC_0805 -> jqi_passives:C_MLCC_0612
- C11: value 10uF -> 10nF; device jqi_passives:C_MLCC_0805 -> jqi_passives:C_MLCC_0306
- C17: value 1uF -> 100nF
- C2, C3: device jqi_passives:C_MLCC_0402 -> jqi_passives:C_MLCC_0603
- C29: value 1uF -> 0.47uF; device jqi_passives:C_MLCC_0603 -> jqi_passives:C_MLCC_0612
- C30, C31: device jqi_passives:C_MLCC_0603 -> jqi_passives:C_MLCC_0306
- CL1, CL2, CL3, CL4, CL5, CL6: value 10nF -> 100nF
- CL12: value 10nF -> 100nF; device jqi_passives:C_MLCC_0402 -> jqi_passives:C_MLCC_0603
- D2: value MMDL770T1G -> Schottky; device zetex:SOD323 -> diode:SOD523
- F3, F4, F7, F8: value (none) -> 1k_ferrite; device jqi_passives:R_0805 -> jqi_passives:L_FERRITE_0603
- IC4: value AD8676 -> MIC5205-5V; device analog-devices:MSOP08 -> regulator-jqi:SOT23-5L
- IC6: value 78L05F -> MIC5205-3V; device linear:SOT89 -> regulator-jqi:SOT23-5L
- MON: value BNC-H -> UMC; device connector-jqi:BNC90 -> connector-jqi:UMC
- MON1: value 50R -> 100R
- R14: value 0R -> (none)
- R15: value 10k -> (none)
- R16: value 3k -> (none)
- R17, R18: value 0R -> 10k
- R19: value 0R -> 28.7k
- R22: value 10k -> 28.7k
- R23: value 10k -> 3k
- RJH1: device jqi_passives:R_0402 -> jqi_passives:R_0603
- moved C29 231.6 mm to (30.0, 19.1), turned to 90 degrees
- moved R15 210.7 mm to (35.2, 31.5)
- moved R18 199.6 mm to (33.8, 64.8), turned to 90 degrees
- moved R16 198.7 mm to (37.1, 48.8), turned to 90 degrees
- moved R14 197.1 mm to (41.1, 36.8), turned to 0 degrees
- moved R17 193.4 mm to (35.4, 64.8), turned to 270 degrees
- moved IC4 189.3 mm to (125.6, 80.4)
- moved C17 175.0 mm to (67.3, 88.0), turned to 180 degrees
- moved IC6 173.6 mm to (65.8, 91.3)
- moved ENC 154.8 mm to (80.3, 80.9), turned to 270 degrees
- moved LCD 153.8 mm to (54.9, 80.9), turned to 270 degrees
- moved R12 144.9 mm to (41.0, 29.1), turned to 90 degrees
- moved R36 144.4 mm to (39.5, 27.6)
- moved R23 144.1 mm to (111.8, 65.0), turned to 180 degrees
- moved F4 143.9 mm to (35.8, 58.9), turned to 90 degrees
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Connections:
- removed net A4: IC5.27, R14.P$2
- removed net A5: IC5.28, R17.P$2
- removed net D10: IC5.14
- removed net D4: IC5.2
- removed net D6: IC5.10
- removed net D7: IC5.11
- removed net N$33: R18.P$1, R23.P$2, R24.P$1
- removed net N$35: JP1.3
- removed net N$46: C11.P$1, C31.P$1, F8.P$2, IC3.11
- removed net N$50: CL1.P$1, CR1.P$1, F6.P$1, IC7.4
- removed net N$52: CL2.P$1, CR2.P$1, F5.P$1, IC7.8
- removed net PC0: IC5.23
- removed net PC1: IC5.24
- removed net PC2: IC5.25
- removed net PC3: IC5.26
- new net +3V: C20.P$1, D3.C, IC6.5, LCD.1, U4.16
- new net -FFWD: FFWD.7, R18.P$2, T1.P$3
- new net DAC_MOSI: IC5.24, R10.P$2
- new net DAC_SCK: IC5.25, R9.P$1
- new net FEED_FWD: JP2.2, MR10.P$1
- new net FFWD: JP3.1, JP3.11, JP3.13, JP3.15, JP3.3, JP3.5, JP3.7, JP3.9, R17.P$1, T1.P$1
- new net FFWD_POSTGAIN: FFWD.1, FFWD.2, JP2.3
- new net GPIO0: J1.A3, JP3.2
- new net GPIO1: J1.C3, JP3.4
- new net GPIO2: J1.A4, JP3.6
- new net GPIO3: J1.C4, JP3.8
- new net GPIO4: J1.A6, JP3.10
- new net GPIO5: J1.C6, JP3.12
- new net GPIO6: J1.A7, JP3.14
- new net GPIO7: J1.C7, JP3.16
- new net LCD_CS_3V: LCD.6, U4.3
- new net LCD_EN: C17.P$1, IC5.9, IC6.3, R25.P$2, U4.13
- new net LCD_MOSI_3V: LCD.3, U4.1
- new net LCD_RST_3V: LCD.8, U4.5
- new net LCD_RS_3V: LCD.7, U4.4
- new net LCD_SCK_3V: LCD.5, U4.2
- new net N$22: R25.P$1, U4.14
- new net VNEG_QUIET: C25.P$1, C26.P$1, C33.P$2, CL2.P$1, CL6.P$1, F7.P$2, FFWD.4, U2.4, U3.4
- new net VPOS_QUIET: C30.P$1, C31.P$1, C32.P$1, CL1.P$1, CL5.P$1, F9.P$2, FFWD.8, U2.8, U3.8
- new net VREG_DAC: C11.P$1, C21.P$1, C22.P$1, C23.P$1, DAC1.3, DAC1.8, F8.P$2
- net A6: now also R19.P$1, R21.P$2; no longer R18.P$2
- net A7: now also D1.C, R22.P$2, R23.P$1; no longer R19.P$2
- net DACG: now also C10.P$2, C11.P$2, C21.P$2, C22.P$2, C23.P$2, R10.P$4, R11.P$3, R9.P$3, U3.6, U3.7; no longer CD3.P$2, CL8.P$2, CR8.P$2, IC7.1, IC7.2, R39.P$1, R43.P$1, R47.P$2
- net DAC_CS: now also IC5.23, R11.P$1; no longer IC5.13, R46.P$2
- net DCLK: now also R9.P$7; no longer R41.P$1
- net DCS: now also R11.P$7; no longer R49.P$2
- net DDATA: now also R10.P$8; no longer R45.P$1
- net ENC_A: now also IC5.14; no longer IC5.32
- net ENC_B: now also IC5.13; no longer IC5.1
- net ENC_SW: now also IC5.32; no longer IC5.12
- net GND: now also C18.P$1, C24.P$2, C25.P$2, C26.P$2, C29.P$2, C32.P$2, C33.P$1, CD1.P$2, CD2.P$2, FFWD.5, JP2.1, L3.P$2, MON.P$2, MON.P$3, R10.P$6, R11.P$5, R13.P$7, R9.P$5, SV2.10, SV2.12, SV2.14, SV2.16, SV2.2, SV2.4, SV2.6, SV2.8; no longer C10.P$2, C11.P$2, C27.P$2, CR1.P$2, CR2.P$2, CR5.P$2, CR6.P$2, D2.2, MON.2, R16.P$2, R24.P$2, R40.P$1, R44.P$1, R48.P$2, R54.P$2, SV2.1, SV2.11, SV2.13, SV2.15, SV2.3, SV2.5, SV2.7, SV2.9
- net LCD_CS: now also IC5.10, U4.10; no longer LCD.6
- net LCD_RS: now also IC5.11, U4.9; no longer LCD.7
- net LCD_RST: now also IC5.12, U4.8; no longer LCD.8
- net MOD_OUT: now also MR10.P$2, MR11.P$2, U2.5; no longer IC4.5
- net MON: now also BUF.1, R13.P$3; no longer BUF1.1, R51.P$1
- net MON_MON: now also MON.P$1; no longer MON.1, R19.P$1
- net MOSI: now also U4.12; no longer LCD.3, R42.P$2
- net N$10: now also U3.1; no longer IC7.7
- net N$12: now also R14.P$1, U3.3; no longer D2.1, R17.P$1, R21.P$2, R22.P$1
- net N$14: now also BUF.2, R13.P$2, R13.P$4; no longer BUF1.2, R51.P$2, R52.P$1
- net N$15: now also R16.P$1, U3.2; no longer BUF1.5, IC7.6
- net N$16: now also R9.P$6, R9.P$8; no longer R40.P$2, R41.P$2
- net N$17: now also BUF.3, R13.P$6, R13.P$8; no longer BUF1.3, R53.P$1, R54.P$1
- net N$18: now also U2.6; no longer IC4.6
- net N$19: now also SV2.1; no longer SV2.2
- net N$2: now also D4.A, JP1.3; no longer JP6.2, R26.P$2
- net N$20: now also MR11.P$1, U2.7; no longer IC4.7
- net N$21: now also C18.P$2, U2.3; no longer IC4.3
- net N$23: now also U2.1; no longer IC4.1
- net N$25: now also U2.2; no longer IC4.2
- net N$27: now also SV2.3; no longer SV2.4
- net N$29: now also R15.P$1, U3.5; no longer R14.P$1, R15.P$2, R16.P$1
- net N$3: now also R11.P$6, R11.P$8; no longer R48.P$1, R49.P$1
- net N$31: now also SV2.5; no longer SV2.6
- net N$34: now also SV2.7; no longer SV2.8
- net N$36: now also BUF.4; no longer BUF1.4
- net N$37: now also BUF.8; no longer BUF1.8
- net N$38: now also FFWD.6, R17.P$2, R18.P$1; no longer C10.P$1, C30.P$1, F7.P$2, IC3.4
- net N$39: now also SV2.9; no longer SV2.10
- net N$4: now also BUF.6, BUF.7, R13.P$1; no longer BUF1.6, BUF1.7, R52.P$2
- net N$40: now also R9.P$2, R9.P$4; no longer R38.P$1, R39.P$2
- net N$41: now also SV2.11; no longer SV2.12
- net N$42: now also R10.P$1, R10.P$3; no longer R42.P$1, R43.P$2
- net N$43: now also SV2.13; no longer SV2.14
- net N$44: now also SV2.15; no longer SV2.16
- net N$47: now also R10.P$5, R10.P$7; no longer R44.P$2, R45.P$2
- net N$48: now also R15.P$2; no longer IC7.3
- net N$49: now also R11.P$2, R11.P$4; no longer R46.P$1, R47.P$1
- net N$6: now also BUF.5, R16.P$2; no longer CL5.P$1, CR5.P$1, F1.P$1, IC4.8
- net N$7: now also FFWD.3, T1.P$2; no longer CL6.P$1, CR6.P$1, F2.P$1, IC4.4
- net N$9: now also R14.P$2; no longer IC7.5
- net SCK: now also U4.11; no longer LCD.5, R38.P$2
- net SW: now also IC5.1
- net V+: now also CD1.P$1, F9.P$1, IC3.4, IC4.1, IC4.3, R19.P$2; no longer F1.P$2, F5.P$2, F7.P$1, IC6.3, R15.P$1
- net V-: now also C24.P$1, CD2.P$1, F7.P$1, IC3.11, R22.P$1; no longer F2.P$2, F6.P$2, F8.P$1, R22.P$2
- net VCC: now also C19.P$1, D2.C, D4.C, IC4.5, R23.P$2; no longer C17.P$1, JP6.1, LCD.1, R21.P$1
- net VREG: now also C10.P$1, F8.P$1, R13.P$5; no longer CD3.P$1, CL8.P$1, CR8.P$1, DAC1.3, DAC1.8, R23.P$1, R53.P$2
- net VREG_EN: now also IC5.2; no longer IC5.9, R26.P$1
- net VSS: now also C19.P$2, C20.P$2, C27.P$2, D1.A, D2.A, D3.A, IC4.2, L3.P$1, R21.P$1, U$5.P$1, U$5.P$10, U$5.P$11, U$5.P$12, U$5.P$13, U$5.P$14, U$5.P$15, U$5.P$16, U$5.P$2, U$5.P$3, U$5.P$4, U$5.P$5, U$5.P$6, U$5.P$7, U$5.P$8, U$5.P$9, U4.15, U4.P$17; no longer C29.P$2, IC6.2@1, JP6.3
Routing:
- net V+: track 1.32 -> 203.5 mm, vias 0 -> 7
- net V-: track 0.00 -> 194.5 mm, vias 0 -> 6
- net FFWD: track 0.00 -> 147.8 mm, vias 0 -> 1
- net VCC: track 1.32 -> 112.4 mm, vias 0 -> 5
- net DAC_CS: track 0.00 -> 85.6 mm, vias 0 -> 2
- net VREG_EN: track 0.00 -> 77.6 mm, vias 0 -> 3
- net DAC_SCK: track 0.00 -> 74.7 mm, vias 0 -> 2
- net DAC_MOSI: track 0.00 -> 69.8 mm, vias 0 -> 2
- net SCK: track 0.00 -> 66.1 mm, vias 0 -> 3
- net MOSI: track 0.00 -> 65.9 mm, vias 0 -> 3
- net VPOS_QUIET: track 0.00 -> 59.1 mm, vias 0 -> 7
- net LCD_EN: track 0.00 -> 53.9 mm
- net VREG: track 0.00 -> 49.4 mm, vias 0 -> 20
- net LCD_RST: track 0.00 -> 45.3 mm
- net LCD_RS: track 0.00 -> 44.0 mm
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- added copper zone on layer 1, net DACG
- added copper zone on layer 15, net DACG
- added copper zone on layer 1, net GND
- added copper zone on layer 15, net GND
- added copper zone on layer 16, net GND
- added copper zone on layer 2, net GND
- added copper zone on layer 16, net VNEG_QUIET
- added copper zone on layer 16, net VPOS_QUIET
- added copper zone on layer 15, net VREG
- added copper zone on layer 1, net VSS
- added copper zone on layer 15, net VSS
- added copper zone on layer 16, net VSS
- added copper zone on layer 2, net VSS
Other:
- board text added: "# 1"
- board text added: "# 2"
- board text added: "# 3"
- board text added: "# 4"
- board text added: "# 5"
- board text added: "# 6"
- board text added: "# 7"
- board text added: "C12-15"
- board text added: "CurrentController v2.0 NCP - 2015"
- board text added: "DCLK"
- board text added: "DCS"
- board text added: "DDATA"
- board text added: "Disabled"
- board text added: "Enabled"
- board text added: "FFW"
- board text added: "FFWD"
- board text added: "Feed Forward"
- board text added: "Feed Forward backplane select"
- board text added: "GPIO # 0"
- board text added: "VNEG_QUIET"
- board text added: "VPOS_QUIET"
- board text added: "VUSB"
- board text removed: "Normal"

Commit message: final routing and gerbers for v2
Parts:
- added IC7: PMOS-SOT323, semiconductor-jqi:SOT323
- added IC8: PMOS-SOT323-SC89, semiconductor-jqi:SC-89
Connections:
- net DC_OUT: now also IC7.3, IC8.P$3
- net N$11: now also IC7.1, IC8.P$1
- net N$15: now also IC7.2, IC8.P$2
Routing:
- net GND: vias 96 -> 135
- added copper zone on layer 1, net N$11
- added copper zone on layer 1, net N$15
Changed lines of the file:
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@@
 <setting verticaltext="up"/>
 </settings>
-<grid distance="0.005" unitdist="inch" unit="inch" style="lines" multiple="1" display="yes" altdistance="0.0005" altunitdist="inch" altunit="inch"/>
+<grid distance="0.001" unitdist="inch" unit="inch" style="lines" multiple="1" display="yes" altdistance="0.0005" altunitdist="inch" altunit="inch"/>
 <layers>
 <layer number="1" name="Top" color="4" fill="1" visible="yes" active="yes"/>
@@
 <text x="63.246" y="25.527" size="0.508" layer="21" rot="R180">DCS</text>
 <text x="27.94" y="50.419" size="0.508" layer="21">VNEG_QUIET</text>
-<text x="31.496" y="25.908" size="0.508" layer="21" rot="R180">VPOS_QUIET</text>
+<text x="32.385" y="25.654" size="0.508" layer="21" rot="R180">VPOS_QUIET</text>
 <text x="7.366" y="35.941" size="0.7112" layer="21">FFW</text>
 <wire x1="16.002" y1="63.627" x2="16.002" y2="81.407" width="0.4064" layer="21"/>
@@
 <text x="25.781" y="90.424" size="1.27" layer="21">CurrentController v2.0
 NCP - 2015</text>
-<text x="52.705" y="42.545" size="1.27" layer="21">C12-15</text>
+<text x="53.594" y="42.672" size="1.27" layer="21">C12-15</text>
 <text x="140.97" y="81.026" size="1.27" layer="21">VUSB</text>
 <text x="112.776" y="54.102" size="1.27" layer="21">ISP Prog</text>
@@
 <elements>
 <element name="CP1" library="rcl" package="PANASONIC_F" value="220uF" x="137.16" y="16.256" smashed="yes" rot="R270">
-<attribute name="NAME" x="139.222" y="16.99" size="0.508" layer="25" rot="R270"/>
+<attribute name="NAME" x="142.27" y="15.593" size="0.508" layer="25" rot="R270"/>
 <attribute name="VALUE" x="134.785" y="18.006" size="1.016" layer="27" rot="R270"/>
 <attribute name="PARTNO" value="PCE3955CT-ND" x="137.16" y="16.256" size="1.778" layer="27" rot="R270" display="off"/>
 </element>
 <element name="CN1" library="rcl" package="PANASONIC_F" value="220uF" x="137.16" y="41.656" smashed="yes" rot="R90">
-<attribute name="NAME" x="135.606" y="41.43" size="0.508" layer="25" rot="R90"/>
+<attribute name="NAME" x="142.845" y="40.033" size="0.508" layer="25" rot="R90"/>
 <attribute name="VALUE" x="139.535" y="39.906" size="1.016" layer="27" rot="R90"/>
 <attribute name="PARTNO" value="PCE3955CT-ND" x="137.16" y="41.656" size="1.778" layer="27" rot="R90" display="off"/>
@@
 </element>
 <element name="IC2" library="misc-ics" package="TO223-3" value="L7912" x="89.662" y="38.1" smashed="yes" rot="R270">
-<attribute name="NAME" x="88.646" y="44.704" size="0.508" layer="25"/>
+<attribute name="NAME" x="88.9" y="44.196" size="0.508" layer="25"/>
 <attribute name="VALUE" x="82.804" y="31.242" size="1.27" layer="27"/>
 <attribute name="PARTNO" value="MC7912CD2TGOS-ND" x="89.662" y="38.1" size="1.778" layer="27" rot="R270" display="off"/>
@@
 <element name="VREFIC" library="linear" package="TO39/4" value="LM399H" x="46.99" y="28.956" smashed="yes" rot="R270">
 <attribute name="PARTNO" value="LM399H#PBF-ND" x="46.99" y="28.956" size="1.778" layer="27" rot="R270" display="off"/>
-<attribute name="NAME" x="44.069" y="22.352" size="1.27" layer="25" ratio="10"/>
+<attribute name="NAME" x="43.688" y="21.971" size="1.27" layer="25" ratio="10"/>
 <attribute name="VALUE" x="46.355" y="32.258" size="1.27" layer="27" ratio="10" rot="R270"/>
 </element>
@@
 </element>
 <element name="C21" library="jqi_passives" package="C_MLCC_0306" value="10nF" x="57.912" y="34.417" smashed="yes" rot="R270">
-<attribute name="NAME" x="58.912" y="35.317" size="1.016" layer="25" font="vector" rot="R270"/>
+<attribute name="NAME" x="59.293" y="35.825" size="1.016" layer="25" font="vector" rot="R270"/>
 <attribute name="PARTNO" value="478-2890-1-ND" x="57.912" y="34.417" size="1.778" layer="27" rot="R270" display="off"/>
 </element>
@@
 <element name="F9" library="jqi_passives" package="L_FERRITE_0603" value="1k_ferrite" x="33.02" y="18.9103" smashed="yes" rot="R90">
 <attribute name="PARTNO" value="490-1034-1-ND" x="27.432" y="15.1003" size="0.508" layer="27" rot="R90" display="off"/>
-<attribute name="NAME" x="35.014" y="18.2183" size="1.016" layer="25" font="vector" rot="R90"/>
+<attribute name="NAME" x="33.363" y="15.8053" size="1.016" layer="25" font="vector" rot="R90"/>
 </element>
 <element name="C29" library="jqi_passives" package="C_MLCC_0612" value="0.47uF" x="29.972" y="19.05" smashed="yes" rot="R90">
 <attribute name="PARTNO" value="490-4382-1-ND" x="33.274" y="19.05" size="0.508" layer="27" rot="R90" display="off"/>
-<attribute name="NAME" x="27.872" y="17.45" size="1.016" layer="25" font="vector" rot="R90"/>
+<attribute name="NAME" x="27.618" y="17.831" size="1.016" layer="25" font="vector" rot="R90"/>
 </element>
 <element name="C30" library="jqi_passives" package="C_MLCC_0306" value="10nF" x="28.448" y="22.606" smashed="yes">
@@
 </element>
 <element name="C31" library="jqi_passives" package="C_MLCC_0306" value="10nF" x="31.496" y="22.606" smashed="yes" rot="R180">
-<attribute name="NAME" x="33.766" y="23.252" size="1.016" layer="25" font="vector" rot="R270"/>
+<attribute name="NAME" x="33.385" y="23.887" size="1.016" layer="25" font="vector" rot="R270"/>
 <attribute name="PARTNO" value="478-2890-1-ND" x="31.496" y="22.606" size="1.778" layer="27" rot="R180" display="off"/>
 </element>
@@
 </element>
 <element name="L3" library="jqi_passives" package="R_0805" value="" x="137.5029" y="92.7354"/>
+<element name="IC8" library="semiconductor-jqi" package="SC-89" value="PMOS-SOT323-SC89" x="36.068" y="44.45" rot="R90"/>
+<element name="IC7" library="semiconductor-jqi" package="SOT323" value="PMOS-SOT323" x="36.068" y="44.45" rot="R90"/>
 </elements>
 <signals>
@@
 <vertex x="0" y="-2.54"/>
 </polygon>
-<via x="76.581" y="23.495" extent="1-16" drill="0.254"/>
+<via x="75.7936" y="24.7142" extent="1-16" drill="0.254"/>
 <wire x1="75.272" y1="17.069" x2="76.149" y2="17.069" width="0.4064" layer="1"/>
 <wire x1="76.149" y1="17.069" x2="76.454" y2="16.764" width="0.4064" layer="1"/>
 <contactref element="L3" pad="P$2"/>
+<via x="8.3566" y="31.6992" extent="1-16" drill="0.254"/>
+<via x="37.3634" y="85.3694" extent="1-16" drill="0.254"/>
+<via x="39.116" y="77.47" extent="1-16" drill="0.254"/>
+<via x="49.1744" y="68.072" extent="1-16" drill="0.254"/>
+<via x="88.4174" y="64.3128" extent="1-16" drill="0.254"/>
+<via x="84.8868" y="49.4538" extent="1-16" drill="0.254"/>
+<via x="112.9792" y="51.308" extent="1-16" drill="0.254"/>
+<via x="128.1684" y="49.8856" extent="1-16" drill="0.254"/>
+<via x="103.7082" y="43.6118" extent="1-16" drill="0.254"/>
+<via x="90.7034" y="45.9486" extent="1-16" drill="0.254"/>
+<via x="52.0446" y="63.1444" extent="1-16" drill="0.254"/>
+<via x="38.2016" y="69.2658" extent="1-16" drill="0.254"/>
+<via x="30.0736" y="60.0456" extent="1-16" drill="0.254"/>
+<via x="15.7226" y="51.7398" extent="1-16" drill="0.254"/>
+<via x="25.1968" y="6.9342" extent="1-16" drill="0.254"/>
+<via x="45.5676" y="9.4488" extent="1-16" drill="0.254"/>
+<via x="56.7436" y="6.6802" extent="1-16" drill="0.254"/>
+<via x="55.3974" y="20.3708" extent="1-16" drill="0.254"/>
+<via x="43.4086" y="18.9484" extent="1-16" drill="0.254"/>
+<via x="78.6892" y="8.7884" extent="1-16" drill="0.254"/>
+<via x="68.4784" y="9.7028" extent="1-16" drill="0.254"/>
+<via x="100.2538" y="6.4516" extent="1-16" drill="0.254"/>
+<via x="118.1862" y="22.8854" extent="1-16" drill="0.254"/>
+<via x="131.8514" y="27.432" extent="1-16" drill="0.254"/>
+<via x="84.1248" y="54.8894" extent="1-16" drill="0.254"/>
+<via x="56.7944" y="69.5706" extent="1-16" drill="0.254"/>
+<via x="43.3832" y="69.1388" extent="1-16" drill="0.254"/>
+<via x="26.1366" y="85.1916" extent="1-16" drill="0.254"/>
+<via x="14.5542" y="62.2808" extent="1-16" drill="0.254"/>
+<via x="11.9634" y="28.8036" extent="1-16" drill="0.254"/>
+<via x="15.6464" y="6.9088" extent="1-16" drill="0.254"/>
+<via x="24.7904" y="15.8242" extent="1-16" drill="0.254"/>
+<via x="138.557" y="94.5134" extent="1-16" drill="0.254"/>
+<via x="139.6238" y="92.9386" extent="1-16" drill="0.254"/>
+<via x="146.05" y="92.1004" extent="1-16" drill="0.254"/>
+<via x="146.4056" y="87.4776" extent="1-16" drill="0.254"/>
+<via x="151.6888" y="92.5322" extent="1-16" drill="0.254"/>
+<via x="148.6916" y="90.805" extent="1-16" drill="0.254"/>
+<via x="143.129" y="93.9546" extent="1-16" drill="0.254"/>
 <wire x1="66.294" y1="45.022" x2="66.944" y2="45.022" width="0" layer="19" extent="1-1"/>
 </signal>
@@
 <wire x1="39.116" y1="43.422" x2="37.168" y2="43.422" width="0.5842" layer="1"/>
 <wire x1="37.168" y1="43.422" x2="37.168" y2="43.5" width="0.5842" layer="1"/>
+<contactref element="IC8" pad="P$1"/>
+<contactref element="IC7" pad="1"/>
+<polygon width="0.127" layer="1" thermals="no">
+<vertex x="36.4236" y="44.196"/>
+<vertex x="36.4236" y="43.053"/>
+<vertex x="37.4904" y="43.053"/>
+<vertex x="37.4904" y="44.196"/>
+</polygon>
 </signal>
 <signal name="N$13">
@@
 <contactref element="R16" pad="P$1"/>
 <wire x1="37.084" y1="48.018" x2="37.084" y2="46.482" width="0.381" layer="1"/>
+<contactref element="IC8" pad="P$2"/>
+<contactref element="IC7" pad="2"/>
+<polygon width="0.127" layer="1" thermals="no">
+<vertex x="36.4236" y="44.704"/>
+<vertex x="36.4236" y="45.847"/>
+<vertex x="37.4396" y="45.847"/>
+<vertex x="37.4396" y="44.7294"/>
+<vertex x="37.4396" y="44.704"/>
+</polygon>
 </signal>
 <signal name="N$4">
@@
 <contactref element="LOUT1" pad="1"/>
 <wire x1="34.968" y1="44.45" x2="28.832" y2="44.45" width="1.016" layer="1"/>
+<contactref element="IC8" pad="P$3"/>
+<contactref element="IC7" pad="3"/>
+<wire x1="35.168" y1="44.45" x2="35.418" y2="44.45" width="0" layer="19" extent="1-1"/>
+<wire x1="34.968" y1="44.45" x2="35.168" y2="44.45" width="0" layer="19" extent="1-1"/>
 </signal>
 <signal name="MOD_OUT">
