File: CurrentController.sch (EAGLE design)
At the start: 135 parts, among them CN1 220uF, CN2 10uF, CN3 47uF, IC1 LM340S-12, IC2 L7912, IC3 TS514, IC4 AD8676, IC5 MEGA8-AI, IC6 78L05F, IC7 AD8676, T1 PVG3A, X1 1-227161-7, X2 1-227161-7, X3 1-227161-7

Commit message: Working on re-routing; about to add feed forward
Parts:
- removed CD7: 100nF, rcl:C-USC0402K
- removed CL10, CL11, CL9: 10nF, rcl:C-USC0402K
- removed CN2, CP2, CR9: 10uF, rcl:C-USC0805K
- removed J2: (no value), 19inch:VG64PD
- removed JP2: (no value), pinhead:PINHD-1X5
- removed JP3: (no value), pinhead:PINHD-1X2
- removed JP4: (no value), pinhead:PINHD-1X7
- removed JP5: (no value), pinhead:PINHD-1X71X07/SMD
- removed LN1, LP1: SDR1005-101K, misc-ics:SDR1005-101K
- removed R10, R25, R9: 10k, rcl:R-US_R0402
- removed R27: 0R, rcl:R-US_R0402
- removed R30, R31, R32, R33, R34, R35: 100R, rcl:R-US_R0402
- removed T1: PVG3A, misc-ics:PVG3A
- removed VREG1: TPS7A470, misc-ics:TPS7A470
- removed X1, X2, X3: 1-227161-7, con-coax:1-227161-7
- added C10, C11, C12, C13, C14, C15, C16: 10uF, jqi_passives:C_MLCC_SMDCMLCC_0805
- added C17: 1uF, jqi_passives:C_MLCC_SMDCMLCC_0603
- added CUR, MOD_IN, MON: BNC-H, connector-jqi:BNC-H
- added D1: Schottky, diode:DIODE-SOD523
- added ENC, LCD: (no value), mcu-accessories:PINHD-2X4-SHROUD
- added F1, F2, F3, F4, F5, F6, F7, F8: (no value), jqi_passives:L_FERRITE_SMDLFERRITE_0805
- added J1: (no value), connector-jqi:VG64C
- added L1, L2: 100uH, jqi_passives:L_FERRITE_SMD-CC1583
- added R6: 0R, jqi_passives:R_SMDR1206
- added U1: TPS7A470, regulator-jqi:TPS7A470
- C1: device rcl:C-USC1206K -> jqi_passives:C_POL_SMDCPOL_1206
- C2, C3, CD3, CL12, CL8: device rcl:C-USC0402K -> jqi_passives:C_MLCC_SMDCMLCC_0402
- C27, C28, C29, CL1, CL2, CL3, CL4, CL5, CL6, MC1: device rcl:C-USC0402K -> jqi_passives:C_MLCC_SMDCMLCC_0603
- C30, C31: value 100nF -> 10nF; device rcl:C-USC0402K -> jqi_passives:C_MLCC_SMDCMLCC_0603
- C4, C5, C6, C7, C8, C9, CR1, CR12, CR2, CR3, CR4, CR5, CR6, CR8: device rcl:C-USC0805K -> jqi_passives:C_MLCC_SMDCMLCC_0805
- MON1, R1, R100, R12, R14, R15, R16, R17, R18, R19, R2, R21, R22, R23, R24, R26, R36, R37, R38, R39, R4, R40, R41, R42, R43, R44, R45, R46, R47, R48, R49, R5, R50, R51, R52, R53, R54: device rcl:R-US_R0402 -> jqi_passives:R_SMDR0603
- MR1, MR2, MR3, MR4, MR5, MR6, MR7, MR8, MR9: device rcl:R-US_R0805 -> jqi_passives:R_SMDR0805
- R20: device rcl:R-US_R0402 -> jqi_passives:R_SMDR0805
- R3, R7, R8: value 10k -> 0R; device rcl:R-US_R0402 -> jqi_passives:R_SMDR1206
- RJH1: value 0R -> 0R_DNP; device rcl:R-US_R0402 -> jqi_passives:R_SMDR0402
- SV2: device con-lstb:MA08-2 -> connector-jqi:MA08-2
Connections:
- net D9 renamed DAC_CS
- net N$6 renamed DC_OUT
- net VOUT renamed MOD_OUT
- removed net +12V: BUF1P.V+, C29.1, C30.1, CL12.1, CL2.1, CL3.1, CL5.1, CR12.1, CR2.1, CR3.1, CR5.1, IC1.VO, IC3P.V+, IC4P.V+, IC6.VI, IC7P.V+, R15.1, VREFIC.3, VREG1.P$15, VREG1.P$16
- removed net +5V: CD7.1, CL9.1, CR9.1, IC5.AVCC, IC5.VCC@1, IC5.VCC@2, IC6.VO, JP5.2, JP6.1, R10.1, R100.2, R21.1, R25.2, R3.1, R9.1, SV1.2
- removed net -12V: BUF1P.V-, C31.1, CL1.1, CL4.1, CL6.1, CR1.1, CR4.1, CR6.1, IC2.VO, IC3P.V-, IC4P.V-, IC7P.V-, R22.2, R37.1, VREFIC.4
- removed net D2: CL10.1, IC5.PD2(INT0), R7.2
- removed net D3: CL11.1, IC5.PD3(INT1), R8.2
- removed net D5: IC5.PD5(T1), R26.1, R27.2
- removed net D8: IC5.PB0(ICP), JP2.4, R10.2
- removed net ENABLE: R27.1, VREG1.P$13
- removed net N$3 (its old number): JP2.1, R7.1, R9.2
- removed net N$5 (its old number): JP2.3, R3.2, R8.1
- removed net N$53: JP4.1, R32.2
- removed net N$54: JP4.2, R33.2
- removed net N$55: JP4.3, R34.2
- removed net N$56: JP4.4, R35.2
- new net CURR_OUT: CUR.1, LOUT1.2, RJH1.1
- new net ENC_A: ENC.8, IC5.PD2(INT0)
- new net ENC_B: ENC.6, IC5.PD3(INT1)
- new net ENC_SW: ENC.4, IC5.PB0(ICP)
- new net LCD_CS: LCD.6
- new net LCD_RS: LCD.7
- new net LCD_RST: LCD.8
- new net N$24: IC2.VI, R3.2
- new net N$26: IC1.VI, R6.2
- new net N$30: CN3.-, L2.2, R3.1, R7.1
- new net N$32: CP3.+, L1.2, R6.1, R8.1
- new net N$37: BUF1P.V+, CL3.1, CR3.1, F3.1
- new net N$50: CL1.1, CR1.1, F6.1, IC7P.V-
- new net N$52: CL2.1, CR2.1, F5.1, IC7P.V+
- new net N$6: CL5.1, CR5.1, F1.1, IC4P.V+
- new net SW: ENC.7
- new net VCC: C17.1, ENC.1, IC5.AVCC, IC5.VCC@1, IC5.VCC@2, IC6.VO, JP6.1, LCD.1, R100.2, R21.1, SV1.2
- new net VREG_EN: IC5.PD5(T1), R26.1, U1.EN
- new net VSS: C17.2, C29.2, ENC.2, IC5.GND, IC5.GND@1, IC5.GND@2, IC6.GND, IC6.GND@1, JP1.1, JP1.2, JP6.3, LCD.2, LCD.4, SV1.6
- net +15V: now also J1.A31, J1.C31, L1.1; no longer CP2.1, J2.A31, J2.C31, LP1.1
- net -15V: now also J1.A30, J1.C30, L2.1; no longer CN2.2, J2.A30, J2.C30, LN1.1
- net D4: no longer JP3.2, R25.1
- net D6: no longer R31.1
- net D7: no longer R30.1
- net GND: now also C1.-, C10.2, C11.2, C12.2, C13.2, C14.2, C15.2, C16.2, CUR.2, J1.A1, J1.C1, MOD_IN.2, MON.2, U1.GND; no longer C1.2, C29.2, CD7.2, CL10.2, CL11.2, CL9.2, CN2.1, CP2.2, CR9.2, IC6.GND, IC6.GND@1, J2.A1, JP1.1, JP1.2, JP2.2, JP2.5, JP3.1, JP4.5, JP4.6, JP4.7, JP5.1, JP5.5, JP5.7, JP6.3, SV1.6, T1.P$1, VREG1.P$7, X1.GND, X3.GND
- net MODIN_B: now also MOD_IN.1; no longer X2.1
- net MON_MON: now also MON.1; no longer X3.1
- net MOSI: now also LCD.3
- net N$19: now also SV2.2, U1.6.4A; no longer SV2.16, VREG1.P$12
- net N$27: now also SV2.4, U1.6.4B; no longer C2.1, VREG1.P$14
- net N$31: now also SV2.6, U1.3.2; no longer SV2.14, VREG1.P$11
- net N$34: now also SV2.8, U1.1.6; no longer SV2.12, VREG1.P$10
- net N$36: now also BUF1P.V-, CL4.1, CR4.1, F4.1; no longer JP5.4, R30.2
- net N$38: now also C10.1, C30.1, F7.2, IC3P.V+; no longer JP5.6, R31.2
- net N$39: now also U1.0.8; no longer VREG1.P$9
- net N$41: now also SV2.12, U1.0.4; no longer SV2.8, VREG1.P$8
- net N$43: now also SV2.14, U1.0.2; no longer SV2.6, VREG1.P$6
- net N$44: now also SV2.16, U1.0.1; no longer SV2.4, VREG1.P$5
- net N$45: now also C2.1, U1.NR; no longer SV2.2, VREG1.P$4
- net N$46: now also C11.1, C31.1, F8.2, IC3P.V-; no longer JP5.3, T1.P$2
- net N$7: now also CL6.1, CR6.1, F2.1, IC4P.V-; no longer LOUT1.2, RJH1.1, X1.1
- net PC0: no longer R35.1
- net PC1: no longer R34.1
- net PC2: no longer R33.1
- net PC3: no longer R32.1
- net SCK: now also LCD.5
- net V+: now also C1.+, C29.1, CL12.1, CR12.1, F1.2, F3.2, F5.2, F7.1, IC1.VO, IC6.VI, R15.1, R8.2, U1.IN, VREFIC.3; no longer CP3.+, IC1.VI, LP1.2
- net V-: now also F2.2, F4.2, F6.2, F8.1, IC2.VO, R22.2, R37.1, R7.2, VREFIC.4; no longer CN3.-, IC2.VI, LN1.2
- net VREG: now also C12.1, C13.1, C14.1, C15.1, C16.1, U1.OUT, U1.SENSE; no longer C1.1, VREG1.P$1, VREG1.P$20, VREG1.P$3
Other:
- note added: "C1 might not be necessary"
- note added: "Check connections"
- note added: "Connect SENSE at load"
- note added: "DACG = VREG - 5V"
- note added: "DNP"
- note added: "For programming, use pullup Use pulldown for normal operation"
- note added: "Model for good decoupling filter?"
- note added: "Mount matching capacitor on reverse side"
- note added: "NEED LEVEL TRANSLATOR"
- note added: "Optional jumper around VREG"
- note added: "RS1, RS2 should be precision resistors, eg, VSMP2010 66R0000ASW"
- note added: "Use: MSS1583-104KE"
- note added: "VCC...? supplied from where? Add diode & can power uC?"
- note added: "additional high-freq capacitor?"
- note added: "caps use C2012X5R1V106K085AC ?"
- note added: "change to resistor array?"
- note added: "mount corresponding cap on reverse side"
- note added: "switch to CoilCraft; use LC filter design tool"
- note removed: ""enable" switch on front panel"
- note removed: "+-12, Vreg"
- note removed: "100uH"
- note removed: "4"
- note removed: "490-2649-1-ND"
- note removed: "5"
- note removed: "6"
- note removed: "7"
- note removed: "CLK"
- note removed: "CS"
- note removed: "Connected to rotary encoder"
- note removed: "DTR"
- note removed: "Data"
- note removed: "E"
- note removed: "Enable for Vreg"
- note removed: "GROUND to get right voltage"
- note removed: "OUT"
- note removed: "RS"
- note removed: "Rot_A -> D2"
- note removed: "Rot_B -> D3"
- note removed: "These should be precision"
- note removed: "VREG_SELECT"
- note removed: "VSMP2010 66R0000ASW"
- note removed: "Vcc"
- note removed: "VregEnable"
- note removed: "add in oscillator"
- note removed: "add jumpers?"
- note removed: "change log: Changed to 2010 resistors!! (7/14/2014)"
- note removed: "connects rotary switch"
- note removed: "contrast"
- note removed: "decouples internal reference"
- note removed: "from op amp"
- note removed: "gnd"
- note removed: "header to rotary encoder switch"
- note removed: "input for enable/disable"
- note removed: "look into how you load bootloader?"
- note removed: "microVcc"
- note removed: "modin_b"
- note removed: "monitor all power supplies with analog in"
- note removed: "or switch - surface mount?"
- note removed: "pin 14"
- note removed: "pin 15"
- note removed: "rotary A"
- note removed: "rotary B"
- note removed: "sense"
- note removed: "test on arduino if IO is pullup on startup"
- note removed: "to op amp"
- note removed: "vout"
- note removed: "vreg"
- moved on the sheet: BUF1A, BUF1B, C2, C27, C28, C29, C3, C30, C31, C4, C5, C6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

Commit message: mostly routed, few remaining tweaks
Parts:
- removed BUF1, IC7: AD8676, analog-devices:AD8656RM
- removed CD3: 100nF, jqi_passives:C_MLCC_SMDCMLCC_0402
- removed CL8: 10nF, jqi_passives:C_MLCC_SMDCMLCC_0402
- removed CR1, CR2, CR5, CR6, CR8: 10uF, jqi_passives:C_MLCC_SMDCMLCC_0805
- removed F1, F2, F5, F6: (no value), jqi_passives:L_FERRITE_SMDLFERRITE_0805
- removed JP6: (no value), pinhead:PINHD-1X3
- removed R24, R26, R38, R39, R40, R41, R42, R43, R44, R45, R46, R47, R48, R49, R51, R52, R53, R54: 10k, jqi_passives:R_SMDR0603
- added BUF, FFWD, U2, U3: AD8676, opamp-jqi:DUAL-OPAMP-AD8676_MSOP
- added C18: (no value), jqi_passives:C_MLCC_SMDCMLCC_0603
- added C19, C20: 1uF, jqi_passives:C_MLCC_SMDCMLCC_0603
- added C21, C25, C26: 10nF, jqi_passives:C_MLCC_SMDCMLCC_0306
- added C22, C23, C32, C33, CD1, CD2: 100nF, jqi_passives:C_MLCC_SMDCMLCC_0603
- added C24: 0.47uF, jqi_passives:C_MLCC_SMDCMLCC_0612
- added D3, D4: Schottky, diode:DIODE-SOD523
- added F9: 1k_ferrite, jqi_passives:L_FERRITE_SMDLFERRITE_0603
- added JP2: (no value), pinhead:PINHD-1X3
- added JP3: (no value), pinhead:PINHD-2X8
- added L3: (no value), jqi_passives:L_FERRITE_SMDLFERRITE_0805
- added MR10, MR11: 1k, jqi_passives:R_SMDR0805
- added R10, R11, R13, R9: 10k, jqi_passives:R_ARRAY
- added R25: 200k, jqi_passives:R_SMDR0603
- added T1: 100k, rlc-jqi:BOURNS-3006P
- added U$5: WURTH_EMI, mcu-accessories:WURTH_EMI
- added U4: NT2006, semiconductor-jqi:NT2006
- C10: value 10uF -> 0.47uF; device jqi_passives:C_MLCC_SMDCMLCC_0805 -> jqi_passives:C_MLCC_SMDCMLCC_0612; PARTNO (none) -> 490-4382-1-ND
- C11: value 10uF -> 10nF; device jqi_passives:C_MLCC_SMDCMLCC_0805 -> jqi_passives:C_MLCC_SMDCMLCC_0306; PARTNO (none) -> 478-2890-1-ND
- C12, C13, C14, C15, C16, CR12, CR3, CR4: PARTNO (none) -> 1276-2890-1-ND
- C17: value 1uF -> 100nF; PARTNO (none) -> 445-1316-1-ND
- C2: device jqi_passives:C_MLCC_SMDCMLCC_0402 -> jqi_passives:C_MLCC_SMDCMLCC_0603; PARTNO (none) -> 1276-1184-1-ND
- C27, C28: PARTNO (none) -> 445-1316-1-ND
- C29: value 1uF -> 0.47uF; device jqi_passives:C_MLCC_SMDCMLCC_0603 -> jqi_passives:C_MLCC_SMDCMLCC_0612; PARTNO (none) -> 490-4382-1-ND
- C3: device jqi_passives:C_MLCC_SMDCMLCC_0402 -> jqi_passives:C_MLCC_SMDCMLCC_0603; PARTNO (none) -> 1276-2119-1-ND
- C30, C31: device jqi_passives:C_MLCC_SMDCMLCC_0603 -> jqi_passives:C_MLCC_SMDCMLCC_0306; PARTNO (none) -> 478-2890-1-ND
- C4, C5, C6, C7, C8, C9: PARTNO (none) -> 445-9112-1-ND
- CL1, CL2, CL3, CL4, CL5, CL6: value 10nF -> 100nF; PARTNO (none) -> 445-1316-1-ND
- CL12: value 10nF -> 100nF; device jqi_passives:C_MLCC_SMDCMLCC_0402 -> jqi_passives:C_MLCC_SMDCMLCC_0603; PARTNO (none) -> 445-1316-1-ND
- CN1, CP1: PARTNO (none) -> PCE3955CT-ND
- CN3, CP3: PARTNO (none) -> 399-3797-1-ND
- D2: value MMDL770T1G -> Schottky; device zetex:DSOD323 -> diode:DIODE-SOD523; PARTNO (none) -> 568-7397-1-ND
- DAC1: PARTNO (none) -> AD5541ARZ-ND
- F3, F4, F7, F8: value (none) -> 1k_ferrite; device jqi_passives:L_FERRITE_SMDLFERRITE_0805 -> jqi_passives:L_FERRITE_SMDLFERRITE_0603; PARTNO (none) -> 490-1034-1-ND
- IC1: PARTNO (none) -> LM340S-12/NOPB-ND
- IC2: PARTNO (none) -> MC7912CD2TGOS-ND
- IC3: PARTNO (none) -> 497-4453-1-ND
- IC4: value AD8676 -> MIC5205-5V; device analog-devices:AD8656RM -> regulator-jqi:MIC5205; PARTNO (none) -> 576-1261-1-ND
- IC6: value 78L05F -> MIC5205-3V; device linear:78L05F -> regulator-jqi:MIC5205; PARTNO (none) -> 576-1258-1-ND
- L1, L2: PARTNO (none) -> MSS1583-104KEB
- LOUT1: PARTNO (none) -> 587-3070-1-ND / DN7906CT-ND
- MC1: PARTNO (none) -> 1276-1184-1-ND
- MON: value BNC-H -> UMC; device connector-jqi:BNC-H -> connector-jqi:UMC
- MON1: value 50R -> 100R; PARTNO (none) -> P100HCT-ND
- MR1, MR2, MR3, MR4, MR5, MR6, MR7, MR8, MR9: PARTNO (none) -> P1.0KBFCT-ND
- QFB1: PARTNO (none) -> NDS0605CT-ND
- R1, R100: PARTNO (none) -> P10.0KHCT-ND
- R12: PARTNO (none) -> P28.7KHCT-ND
- R14: value 0R -> (none)
- R15: value 10k -> (none)
- R16: value 3k -> (none)
- R17, R18: value 0R -> 10k; PARTNO (none) -> P10.0KHCT-ND
- R19: value 0R -> 28.7k; PARTNO (none) -> P28.7KHCT-ND
- R2: PARTNO (none) -> P100HCT-ND
- R21, R4, R5, R50: PARTNO (none) -> P3.00KHCT-ND
- R22: value 10k -> 28.7k; PARTNO (none) -> P28.7KHCT-ND
- R23: value 10k -> 3k; PARTNO (none) -> P3.00KHCT-ND
- R3, R6, R7, R8: PARTNO (none) -> P0.0ECT-ND
- R36: PARTNO (none) -> P11.0KHCT-ND
- R37: PARTNO (none) -> P7.50KHCT-ND
- RJH1: device jqi_passives:R_SMDR0402 -> jqi_passives:R_SMDR0603
- U1: PARTNO (none) -> 296-37243-1-ND
- VREFIC: PARTNO (none) -> LM399H#PBF-ND
Connections:
- removed net A4: IC5.PC4(ADC4/SDA), R14.2
- removed net A5: IC5.PC5(ADC5/SCL), R17.2
- removed net D10: IC5.PB2(SS/OC1B)
- removed net D4: IC5.PD4(XCK/T0)
- removed net D6: IC5.PD6(AIN0)
- removed net D7: IC5.PD7(AIN1)
- removed net N$33: R18.1, R23.2, R24.1
- removed net N$35: JP1.3
- removed net N$46: C11.1, C31.1, F8.2, IC3P.V-
- removed net N$50: CL1.1, CR1.1, F6.1, IC7P.V-
- removed net N$52: CL2.1, CR2.1, F5.1, IC7P.V+
- removed net PC0: IC5.PC0(ADC0)
- removed net PC1: IC5.PC1(ADC1)
- removed net PC2: IC5.PC2(ADC2)
- removed net PC3: IC5.PC3(ADC3)
- new net +3V: C20.1, D3.C, IC6.OUT, LCD.1, U4.VA
- new net -FFWD: FFWDB.OUT, R18.2, T1.P$3
- new net DAC_MOSI: IC5.PC1(ADC1), R10A.2
- new net DAC_SCK: IC5.PC2(ADC2), R9A.1
- new net FEED_FWD: JP2.2, MR10.1
- new net FFWD: JP3.1, JP3.11, JP3.13, JP3.15, JP3.3, JP3.5, JP3.7, JP3.9, R17.1, T1.P$1
- new net FFWD_POSTGAIN: FFWDA.-IN, FFWDA.OUT, JP2.3
- new net GPIO0: J1.A3, JP3.2
- new net GPIO1: J1.C3, JP3.4
- new net GPIO2: J1.A4, JP3.6
- new net GPIO3: J1.C4, JP3.8
- new net GPIO4: J1.A6, JP3.10
- new net GPIO5: J1.C6, JP3.12
- new net GPIO6: J1.A7, JP3.14
- new net GPIO7: J1.C7, JP3.16
- new net LCD_CS_3V: LCD.6, U4.A3
- new net LCD_EN: C17.1, IC5.PD5(T1), IC6.EN, R25.2, U4.VB
- new net LCD_MOSI_3V: LCD.3, U4.A1
- new net LCD_RST_3V: LCD.8, U4.A5
- new net LCD_RS_3V: LCD.7, U4.A4
- new net LCD_SCK_3V: LCD.5, U4.A2
- new net N$22: R25.1, U4.EN
- new net VNEG_QUIET: C25.1, C26.1, C33.2, CL2.1, CL6.1, F7.2, FFWDP.V-, U2P.V-, U3P.V-
- new net VPOS_QUIET: C30.1, C31.1, C32.1, CL1.1, CL5.1, F9.2, FFWDP.V+, U2P.V+, U3P.V+
- new net VREG_DAC: C11.1, C21.1, C22.1, C23.1, DAC1.REF, DAC1.VDD, F8.2
- net A6: now also R19.1, R21.2; no longer R18.2
- net A7: now also D1.C, R22.2, R23.1; no longer R19.2
- net DACG: now also C10.2, C11.2, C21.2, C22.2, C23.2, R10B.2, R11B.1, R9B.1, U3B.-IN, U3B.OUT; no longer CD3.2, CL8.2, CR8.2, IC7A.IN-, IC7A.OUT, R39.1, R43.1, R47.2
- net DAC_CS: now also IC5.PC0(ADC0), R11A.1; no longer IC5.PB1(OC1A), R46.2
- net DCLK: now also R9D.1; no longer R41.1
- net DCS: now also R11D.1; no longer R49.2
- net DDATA: now also R10D.2; no longer R45.1
- net ENC_A: now also IC5.PB2(SS/OC1B); no longer IC5.PD2(INT0)
- net ENC_B: now also IC5.PB1(OC1A); no longer IC5.PD3(INT1)
- net ENC_SW: now also IC5.PD2(INT0); no longer IC5.PB0(ICP)
- net GND: now also C18.1, C24.2, C25.2, C26.2, C29.2, C32.2, C33.1, CD1.2, CD2.2, FFWDB.+IN, JP2.1, L3.2, R10C.2, R11C.1, R13D.1, R9C.1, SV2.10, SV2.12, SV2.14, SV2.16, SV2.2, SV2.4, SV2.6, SV2.8; no longer C10.2, C11.2, C27.2, CR1.2, CR2.2, CR5.2, CR6.2, D2.A, R16.2, R24.2, R40.1, R44.1, R48.2, R54.2, SV2.1, SV2.11, SV2.13, SV2.15, SV2.3, SV2.5, SV2.7, SV2.9
- net LCD_CS: now also IC5.PD6(AIN0), U4.B3; no longer LCD.6
- net LCD_RS: now also IC5.PD7(AIN1), U4.B4; no longer LCD.7
- net LCD_RST: now also IC5.PB0(ICP), U4.B5; no longer LCD.8
- net MOD_OUT: now also MR10.2, MR11.2, U2B.+IN; no longer IC4B.IN+
- net MON: now also BUFA.OUT, R13B.1; no longer BUF1A.OUT, R51.1
- net MON_MON: no longer R19.1
- net MOSI: now also U4.B1; no longer LCD.3, R42.2
- net N$10: now also U3A.OUT; no longer IC7B.OUT
- net N$12: now also R14.1, U3A.+IN; no longer D2.C, R17.1, R21.2, R22.1
- net N$14: now also BUFA.-IN, R13A.2, R13B.2; no longer BUF1A.IN-, R51.2, R52.1
- net N$15: now also R16.1, U3A.-IN; no longer BUF1B.IN+, IC7B.IN-
- net N$16: now also R9C.2, R9D.2; no longer R40.2, R41.2
- net N$17: now also BUFA.+IN, R13C.2, R13D.2; no longer BUF1A.IN+, R53.1, R54.1
- net N$18: now also U2B.-IN; no longer IC4B.IN-
- net N$19: now also SV2.1; no longer SV2.2
- net N$2: now also D4.A, JP1.3; no longer JP6.2, R26.2
- net N$20: now also MR11.1, U2B.OUT; no longer IC4B.OUT
- net N$21: now also C18.2, U2A.+IN; no longer IC4A.IN+
- net N$23: now also U2A.OUT; no longer IC4A.OUT
- net N$25: now also U2A.-IN; no longer IC4A.IN-
- net N$27: now also SV2.3; no longer SV2.4
- net N$29: now also R15.1, U3B.+IN; no longer R14.1, R15.2, R16.1
- net N$3: now also R11C.2, R11D.2; no longer R48.1, R49.1
- net N$31: now also SV2.5; no longer SV2.6
- net N$34: now also SV2.7; no longer SV2.8
- net N$36: now also BUFP.V-; no longer BUF1P.V-
- net N$37: now also BUFP.V+; no longer BUF1P.V+
- net N$38: now also FFWDB.-IN, R17.2, R18.1; no longer C10.1, C30.1, F7.2, IC3P.V+
- net N$39: now also SV2.9; no longer SV2.10
- net N$4: now also BUFB.-IN, BUFB.OUT, R13A.1; no longer BUF1B.IN-, BUF1B.OUT, R52.2
- net N$40: now also R9A.2, R9B.2; no longer R38.1, R39.2
- net N$41: now also SV2.11; no longer SV2.12
- net N$42: now also R10A.1, R10B.1; no longer R42.1, R43.2
- net N$43: now also SV2.13; no longer SV2.14
- net N$44: now also SV2.15; no longer SV2.16
- net N$47: now also R10C.1, R10D.1; no longer R44.2, R45.2
- net N$48: now also R15.2; no longer IC7A.IN+
- net N$49: now also R11A.2, R11B.2; no longer R46.1, R47.1
- net N$6: now also BUFB.+IN, R16.2; no longer CL5.1, CR5.1, F1.1, IC4P.V+
- net N$7: now also FFWDA.+IN, T1.P$2; no longer CL6.1, CR6.1, F2.1, IC4P.V-
- net N$9: now also R14.2; no longer IC7B.IN+
- net SCK: now also U4.B2; no longer LCD.5, R38.2
- net SW: now also IC5.PD3(INT1)
- net V+: now also CD1.1, F9.1, IC3P.V+, IC4.EN, IC4.IN, R19.2; no longer F1.2, F5.2, F7.1, IC6.VI, R15.1
- net V-: now also C24.1, CD2.1, F7.1, IC3P.V-, R22.1; no longer F2.2, F6.2, F8.1, R22.2
- net VCC: now also C19.1, D2.C, D4.C, IC4.OUT, IC6.IN, R23.2; no longer C17.1, IC6.VO, JP6.1, LCD.1, R21.1
- net VREG: now also C10.1, F8.1, R13C.1; no longer CD3.1, CL8.1, CR8.1, DAC1.REF, DAC1.VDD, R23.1, R53.2
- net VREG_EN: now also IC5.PD4(XCK/T0); no longer IC5.PD5(T1), R26.1
- net VSS: now also C19.2, C20.2, C27.2, D1.A, D2.A, D3.A, IC4.GND, L3.1, R21.1, U$5.GND, U4.GND; no longer C29.2, IC6.GND@1, JP6.3
Other:
- note added: "+5V"
- note added: "BUF1A re-centers output around GND; Using same resistor array (+/- 5%) as for digital comm op amps, at most introduces slight nonlinearity to monitor signal but much cheaper/simpler."
- note added: "CHECK IF NEED ADDITIONAL Volt Stepdown?"
- note added: "CHECK PACKAGE!!"
- note added: "FFW signal from backplane"
- note added: "I think this should work ok, but needs testing."
- note added: "POT controls gain between +/- 1. CW motion = decreasing gain. Note: Polarity inversion @ G = 0."
- note added: "Short beneath this component"
- note added: "Short here, might solder in?"
- note added: "To go around uC"
- note added: "V+ mon"
- note added: "V- mon"
- note added: "change MR5 val; figure out C18 val"
- note added: "feed forward"
- note added: "monitor for +/-V"
- note added: "short here; solder later?"
- note removed: "+12V monitor"
- note removed: "100mA, 5V"
- note removed: "A4"
- note removed: "A5"
- note removed: "A6"
- note removed: "A7"
- note removed: "For programming, use pullup Use pulldown for normal operation"
- note removed: "NEED LEVEL TRANSLATOR"
- note removed: "PC0"
- note removed: "PC1"
- note removed: "PC2"
- note removed: "PC3"
- note removed: "RXI"
- note removed: "TXO"
- note removed: "VCC...? supplied from where? Add diode & can power uC?"
- note removed: "caps use C2012X5R1V106K085AC ?"
- note removed: "change to resistor array?"
- note removed: "enable Switch"
- note removed: "monitor voltage levels"

Commit message: final routing and gerbers for v2
Parts:
- added IC7: PMOS-SOT323, semiconductor-jqi:PMOS-SOT323
- added IC8: PMOS-SOT323-SC89, semiconductor-jqi:PMOS-SOT323-SC89
Connections:
- net DC_OUT: now also IC7.D, IC8.D
- net N$11: now also IC7.G, IC8.G
- net N$15: now also IC7.S, IC8.S
Other:
- note added: "Temp packages, to decide on right MOS"
Changed lines of the file:
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@@
 <part name="VSS12" library="supply1" deviceset="VSS" device=""/>
 <part name="GND19" library="supply1" deviceset="GND" device=""/>
+<part name="IC8" library="semiconductor-jqi" deviceset="PMOS-SOT323" device="-SC89"/>
+<part name="IC7" library="semiconductor-jqi" deviceset="PMOS-SOT323" device=""/>
 </parts>
 <sheets>
@@
 <text x="35.56" y="330.2" size="1.778" layer="98" rot="R90">Short beneath this component</text>
 <text x="-17.78" y="210.82" size="1.778" layer="91">CHECK PACKAGE!!</text>
+<text x="20.32" y="279.4" size="1.778" layer="91">Temp packages, to decide on right MOS</text>
 </plain>
 <instances>
@@
 </instance>
 <instance part="MON" gate="G$1" x="-5.08" y="208.28" rot="MR0"/>
+<instance part="IC8" gate="G$1" x="40.64" y="248.92"/>
+<instance part="IC7" gate="G$1" x="40.64" y="266.7"/>
 </instances>
 <busses>
@@
 <pinref part="QFB1" gate="G$1" pin="G"/>
 <wire x1="-48.26" y1="238.76" x2="-35.56" y2="238.76" width="0.1524" layer="91"/>
+</segment>
+<segment>
+<pinref part="IC8" gate="G$1" pin="G"/>
+<wire x1="35.56" y1="246.38" x2="30.48" y2="246.38" width="0.1524" layer="91"/>
+<wire x1="30.48" y1="246.38" x2="27.94" y2="246.38" width="0.1524" layer="91"/>
+<wire x1="35.56" y1="264.16" x2="30.48" y2="264.16" width="0.1524" layer="91"/>
+<wire x1="30.48" y1="264.16" x2="30.48" y2="246.38" width="0.1524" layer="91"/>
+<junction x="30.48" y="246.38"/>
+<label x="25.4" y="264.16" size="1.778" layer="95"/>
+<pinref part="IC7" gate="G$1" pin="G"/>
 </segment>
 </net>
@@
 <pinref part="R16" gate="G$1" pin="1"/>
 <wire x1="-147.32" y1="223.52" x2="-147.32" y2="226.06" width="0.1524" layer="91"/>
+</segment>
+<segment>
+<pinref part="IC8" gate="G$1" pin="S"/>
+<wire x1="40.64" y1="238.76" x2="40.64" y2="241.3" width="0.1524" layer="91"/>
+<wire x1="40.64" y1="241.3" x2="40.64" y2="243.84" width="0.1524" layer="91"/>
+<wire x1="40.64" y1="261.62" x2="48.26" y2="261.62" width="0.1524" layer="91"/>
+<wire x1="48.26" y1="261.62" x2="48.26" y2="241.3" width="0.1524" layer="91"/>
+<wire x1="48.26" y1="241.3" x2="40.64" y2="241.3" width="0.1524" layer="91"/>
+<junction x="40.64" y="241.3"/>
+<label x="40.64" y="238.76" size="1.778" layer="95"/>
+<pinref part="IC7" gate="G$1" pin="S"/>
 </segment>
 </net>
@@
 <wire x1="1.27" y1="382.27" x2="-10.16" y2="382.27" width="0.1524" layer="91"/>
 </segment>
-</net>
+<segment>
+<pinref part="IC8" gate="G$1" pin="D"/>
+<wire x1="40.64" y1="254" x2="45.72" y2="254" width="0.1524" layer="91"/>
+<wire x1="45.72" y1="254" x2="45.72" y2="274.32" width="0.1524" layer="91"/>
+<wire x1="45.72" y1="274.32" x2="40.64" y2="274.32" width="0.1524" layer="91"/>
+<wire x1="40.64" y1="274.32" x2="40.64" y2="271.78" width="0.1524" layer="91"/>
+<label x="40.64" y="274.32" size="1.778" layer="95"/>
+<pinref part="IC7" gate="G$1" pin="D"/>
+</segment>
+</net>
